Commit message: Update 25.04 -- many changes

File: dev_ws/src/minirys_sim/description/camera.xacro (robot description, xacro)
@@ -21,10 +21,14 @@
             </geometry>
         </collision>
-        <inertial>
+        <!-- <inertial>
             <origin xyz="0 0 0" rpy="0 0 0"/>
             <mass value="0.00003215"/>
-            <inertia ixx="0.00002345" ixy="0.00000000" ixz="0.00000038"
-                     iyy="0.00002166" iyz="0.00000000" izz="0.00001207"/>
-        </inertial>
+            <inertia ixx="0.00002345"
+                     ixy="0.00000000"
+                     ixz="0.00000038"
+                     iyy="0.00002166"
+                     iyz="0.00000000"
+                     izz="0.00001207"/>
+        </inertial> -->
     </link>
     <gazebo reference="bumper">
@@ -56,8 +60,8 @@
         <visual>
             <material>
-                <script>
-                    <uri>${rys_materials_path}</uri>
-                    <name>${gazebo_camera_base_material}</name>
-                </script>
+                <ambient>0.20 0.20 0.20</ambient>
+                <diffuse>0.20 0.20 0.20</diffuse>
+                <specular>0.40 0.40 0.40 1.00 5.00</specular>
+                <emissive>0 0 0 1</emissive>
             </material>
         </visual>
@@ -113,8 +117,8 @@
         <visual>
             <material>
-                <script>
-                    <uri>${rys_materials_path}</uri>
-                    <name>${gazebo_camera_PCB_material}</name>
-                </script>
+                <ambient>0.10 0.10 0.10</ambient>
+                <diffuse>0.10 0.10 0.10</diffuse>
+                <specular>0.40 0.40 0.40 1.00 5.00</specular>
+                <emissive>0 0 0 1</emissive>
             </material>
         </visual>
@@ -138,8 +142,8 @@
         <visual>
             <material>
-                <script>
-                    <uri>${rys_materials_path}</uri>
-                    <name>rys/lens</name>
-                </script>
+                <ambient>0.75 0.75 0.8</ambient>
+                <diffuse>0.75 0.75 0.8</diffuse>
+                <specular>0.75 0.75 0.8 0.3 5</specular>
+                <emissive>0 0 0 1</emissive>
             </material>
         </visual>

File: dev_ws/src/minirys_sim/description/chassis.xacro (robot description, xacro)
@@ -2,12 +2,5 @@
 <robot xmlns:xacro="http://www.ros.org/wiki/xacro">
     <!-- BASE LINK -->
-        <!-- <link name="base_footprint"></link> -->
         <link name="base_link"></link>
-        <!-- <joint name="base_footprint_joint" type="fixed">
-            <parent link="base_link"/>
-            <child link="base_footprint"/>
-            <origin xyz="0 0 -${wheel_radius}"/>
-        </joint>
-     -->
     <!-- SKELETON LINK -->
         <joint name="chassis_joint" type="fixed">
@@ -26,8 +19,24 @@
             <!-- COLISION -->
             <collision name='chassis_box'>
-                <origin xyz="0 0 0.0385" rpy="0 0 0"/>
+                <origin xyz="0 0 0.03515" rpy="0 0 0"/>
                 <geometry>
-                    <box size="0.07 0.116 0.13"/>
+                    <box size="0.07 0.116 0.12"/>
                 </geometry>
+                <surface>
+                    <friction>
+                        <bounce>
+                            <restitution_coefficient>0</restitution_coefficient>
+                            <threshold>1e+06</threshold>
+                        </bounce>
+                      <ode>
+                        <mu>$(arg chassis_mu1)</mu>
+                        <mu2>$(arg chassis_mu2)</mu2>
+                        <kp>$(arg chassis_kp)</kp>
+                        <kd>$(arg chassis_kd)</kd>
+                        <slip1>1.0</slip1>
+                        <slip2>1.0</slip2>
+                      </ode>
+                    </friction>
+                  </surface>
             </collision>
             <collision name='side_bumper'>
@@ -35,4 +44,32 @@
                 <geometry>
                     <cylinder radius="0.056" length="0.01"/>
+                </geometry>
+                <surface>
+                    <friction>
+                        <bounce>
+                            <restitution_coefficient>0</restitution_coefficient>
+                            <threshold>1e+06</threshold>
+                        </bounce>
+                      <ode>
+                        <mu>$(arg chassis_mu1)</mu>
+                        <mu2>$(arg chassis_mu2)</mu2>
+                        <kp>$(arg chassis_kp)</kp>
+                        <kd>$(arg chassis_kd)</kd>
+                        <slip1>1.0</slip1>
+                        <slip2>1.0</slip2>
+                      </ode>
+                    </friction>
+                  </surface>
+            </collision>
+            <collision name='front_battery'>
+                <origin xyz="0.036 0 0" rpy="${pi/2} 0 0"/>
+                <geometry>
+                    <cylinder radius="0.01" length="0.071"/>
+                </geometry>
+            </collision>
+            <collision name='back_battery'>
+                <origin xyz="-0.038 0 0" rpy="${pi/2} 0 0"/>
+                <geometry>
+                    <cylinder radius="0.01" length="0.071"/>
                 </geometry>
             </collision>
@@ -44,8 +81,12 @@
             </collision>
             <inertial>
-                <origin xyz="0 0 0" rpy="0 0 0"/>
-                <mass value="0.75202927"/>
-                <inertia ixx="0.00149038" ixy="-0.00000016" ixz="0.00000155"
-                         iyy="0.00084463" iyz="-0.00000170" izz="0.00108896"/>
+                <origin xyz="$(arg chassis_mx) $(arg chassis_my) $(arg chassis_mz)" rpy="0 0 0"/>
+                <mass value="1.75203002"/>
+                <inertia ixx="$(arg chassis_ixx)"
+                         ixy="$(arg chassis_ixy)"
+                         ixz="$(arg chassis_ixz)"
+                         iyy="$(arg chassis_iyy)"
+                         iyz="$(arg chassis_iyz)"
+                         izz="$(arg chassis_izz)"/>
             </inertial>
         </link>
@@ -53,16 +94,21 @@
             <visual>
                 <material>
-                    <script>
-                        <uri>${rys_materials_path}</uri>
-                        <name>${gazebo_skeleton_material}</name>
-                    </script>
+                        <ambient>0.10 0.10 0.10</ambient>
+                        <diffuse>0.10 0.10 0.10</diffuse>
+                        <specular>0.40 0.40 0.40 1.00 5.00</specular>
+                        <emissive>0 0 0 1</emissive>
                 </material>
             </visual>
+            <!-- <soft_cfm>0</soft_cfm>
+            <soft_erp>0.2</soft_erp> -->
             <mu1>$(arg chassis_mu1)</mu1>
             <mu2>$(arg chassis_mu2)</mu2>
             <kp>$(arg chassis_kp)</kp>
             <kd>$(arg chassis_kd)</kd>
+            <slip1>1.0</slip1>
+            <slip2>1.0</slip2>
+            <fdir1 value="0 0 1"/>
             <selfCollide>false</selfCollide>
-            <gravity>true</gravity>
+            <!-- <gravity>true</gravity> -->
         </gazebo>
     <!-- VISUAL LINKS -->
@@ -110,8 +156,8 @@
             <visual>
                 <material>
-                    <script>
-                        <uri>${rys_materials_path}</uri>
-                        <name>${gazebo_internal_components_material}</name>
-                    </script>
+                    <ambient>0.50 0.50 0.50</ambient>
+                    <diffuse>0.75 0.75 0.75</diffuse>
+                    <specular>0.90 0.90 0.90 50.00 50.00</specular>
+                    <emissive>0 0 0 1</emissive>
                 </material>
             </visual>
@@ -135,8 +181,8 @@
             <visual>
                 <material>
-                    <script>
-                        <uri>${rys_materials_path}</uri>
-                        <name>${gazebo_batteries_material}</name>
-                    </script>
+                    <ambient>0.40 0.00 0.80</ambient>
+                    <diffuse>0.00 0.00 0.50</diffuse>
+                    <specular>0.40 0.40 0.40 1.00 5.00</specular>
+                    <emissive>0 0 0 1</emissive>
                 </material>
             </visual>

File: dev_ws/src/minirys_sim/description/diff_control.xacro (robot description, xacro)
@@ -12,6 +12,6 @@
             <wheel_separation>${wheel_separation}</wheel_separation>
             <wheel_diameter>${wheel_radius*2}</wheel_diameter>
-            <max_wheel_torque>5</max_wheel_torque>
-            <max_wheel_acceleration>10.0</max_wheel_acceleration>
+            <max_wheel_torque>2.5</max_wheel_torque>
+            <max_wheel_acceleration>2.0</max_wheel_acceleration>
             <publish_odom>1</publish_odom>
             <publish_odom_tf>1</publish_odom_tf>

File: dev_ws/src/minirys_sim/description/label.xacro (robot description, xacro)
@@ -13,5 +13,5 @@
                     <box size="0.0001 $(arg label_x) $(arg label_y)"/>
             </geometry>
-            <material name="rys/white"/>
+            <material name="white"/>
         </visual>
     </link>

File: dev_ws/src/minirys_sim/description/macros.xacro (robot description, xacro)
@@ -1,5 +1,5 @@
 <?xml version="1.0"?>
 <robot xmlns:xacro="http://www.ros.org/wiki/xacro">
-    <xacro:macro name="gazebo_single_tof_sensor" params="frame name on visible material">
+    <xacro:macro name="gazebo_single_tof_sensor" params="frame name on visible">
         <gazebo reference="${frame}">
             <sensor name="${name}" type="ray">
@@ -34,5 +34,5 @@
                     </noise>
                 </ray>
-                <plugin name="gazebo_ray" filename="libgazebo_ros_ray_sensor.so">
+                <plugin name="${name}_gazebo_ray" filename="libgazebo_ros_ray_sensor.so">
                     <ros>
                         <namespace>/$(arg robot_namespace)/distance</namespace>
@@ -47,6 +47,8 @@
                 <material>
                     <script>
-                        <uri>${rys_materials_path}</uri>
-                        <name>${material}</name>
+                        <ambient>1.00 0.20 0.20</ambient>
+                        <diffuse>0.60 0.00 0.00</diffuse>
+                        <specular>0.40 0.40 0.40 1.00 5.00</specular>
+                        <emissive>0 0 0 1</emissive>
                     </script>
                 </material>

File: dev_ws/src/minirys_sim/description/materials.xacro (robot description, xacro)
@@ -19,4 +19,7 @@
         <color rgba="0.100000 0.100000 0.100000 1.000000"/>
     </material>
+    <material name="white">
+        <color rgba="0.900000 0.900000 0.900000 1.000000"/>
+    </material>
     <material name="lens">
         <color rgba="0.750000 0.750000 0.800000 0.500000"/>

File: dev_ws/src/minirys_sim/description/robot.urdf.xacro (robot description, xacro)
@@ -15,10 +15,20 @@
             <xacro:arg name="vertical_sensor_visibility" default="false"/>
             <xacro:arg name="all_sensor_visibility" default="false"/>
-            <xacro:arg name="none_sensor_visibility" default="true"/>
-        <!-- PHYSICS -->
+        <!-- CHASSIS PHYSICS -->
         <xacro:arg name="chassis_mu1" default="0.1"/> <!--SURFACE FRICTION-->
         <xacro:arg name="chassis_mu2" default="0.1"/> <!--SURFACE FRICTION-->
         <xacro:arg name="chassis_kp" default="0.7"/>  <!--STIFFNESS-->
         <xacro:arg name="chassis_kd" default="0.05"/> <!--DAMPING-->
+            <!-- CHASSIS INERTIA -->
+            <xacro:arg name="chassis_mx" default="0.000001"/>
+            <xacro:arg name="chassis_my" default="0.000109"/>
+            <xacro:arg name="chassis_mz" default="0.011152"/>
+            <xacro:arg name="chassis_ixx" default="0.00149038"/>
+            <xacro:arg name="chassis_ixy" default="-0.00000016"/>
+            <xacro:arg name="chassis_ixz" default="0.00000155"/>
+            <xacro:arg name="chassis_iyy" default="0.00084463"/>
+            <xacro:arg name="chassis_iyz" default="-0.00000170"/>
+            <xacro:arg name="chassis_izz" default="0.00108896"/>
+        <!-- WHEELS PHYSICS -->
         <xacro:arg name="wheel_mu1" default="10"/>    <!--SURFACE FRICTION-->
         <xacro:arg name="wheel_mu2" default="10"/>    <!--SURFACE FRICTION-->
@@ -27,5 +37,12 @@
         <xacro:arg name="wheel_joint_dumping" default="0.01"/> <!--JOINT DAMPING-->
         <xacro:arg name="wheel_joint_friction" default="0.1"/> <!--JOINT FRICTION-->
-        <!-- ROS -->
+            <!-- CHASSIS INERTIA -->
+            <xacro:arg name="wheels_ixx" default="0.00006281"/>
+            <xacro:arg name="wheels_ixy" default="0.0"/>
+            <xacro:arg name="wheels_ixz" default="0.0"/>
+            <xacro:arg name="wheels_iyy" default="0.00006281"/>
+            <xacro:arg name="wheels_iyz" default="0.0"/>
+            <xacro:arg name="wheels_izz" default="0.00011530"/>
+            <!-- ROS -->
         <xacro:arg name="robot_namespace" default="robot"/>
         <xacro:arg name="package_path" default=""/>
@@ -34,7 +51,6 @@
         <xacro:arg name="vertical_sensor_visibility" default="false"/>
         <xacro:arg name="all_sensor_visibility" default="false"/>
-        <xacro:arg name="none_sensor_visibility" default="true"/>
         <xacro:arg name="camera_visibility" default="false"/>
-        <xacro:arg name="camera_enabled" default="true"/>
+        <xacro:arg name="camera_enabled" default="True"/>
         <xacro:arg name="TOF_FOV_angle" default="0.001"/> <!--FOV - Field of View-->
         <xacro:arg name="TOF_range" default="2"/>
@@ -47,5 +63,4 @@
             <xacro:include filename="macros.xacro"/>
         <!-- ROBOT -->
-            <!-- <xacro:include filename="ros2_control_gazebo.xacro"/> -->
             <xacro:include filename="diff_control.xacro"/>
             <xacro:include filename="chassis.xacro"/>

File: dev_ws/src/minirys_sim/description/tof_sensors.xacro (robot description, xacro)
@@ -19,6 +19,5 @@
                                     name="upper_tof"
                                     on="true"
-                                    visible="${up_down_sensor_visibility}"
-                                    material="${gazebo_tof_material}"/>
+                                    visible="${up_down_sensor_visibility}"/>
     <!-- LOWER SENSOR -->
     <joint name="lower_tof_joint" type="fixed">
@@ -39,6 +38,5 @@
                                     name="lower_tof"
                                     on="true"
-                                    visible="${up_down_sensor_visibility}"
-                                    material="${gazebo_tof_material}"/>
+                                    visible="${up_down_sensor_visibility}"/>
     <!-- LEFT SENSOR -->
     <joint name="left_tof_joint" type="fixed">
@@ -59,6 +57,5 @@
                                     name="left_tof"
                                     on="true"
-                                    visible="${right_left_sensor_visibility}"
-                                    material="${gazebo_tof_material}"/>
+                                    visible="${right_left_sensor_visibility}"/>
     <!-- RIGHT SENSOR -->
     <joint name="right_tof_joint" type="fixed">
@@ -79,6 +76,5 @@
                                     name="right_tof"
                                     on="true"
-                                    visible="${right_left_sensor_visibility}"
-                                    material="${gazebo_tof_material}"/>
+                                    visible="${right_left_sensor_visibility}"/>
     <!-- FRONT SENSOR -->
     <joint name="front_tof_joint" type="fixed">
@@ -99,6 +95,5 @@
                                     name="front_tof"
                                     on="true"
-                                    visible="${front_back_sensor_visibility}"
-                                    material="${gazebo_tof_material}"/>
+                                    visible="${front_back_sensor_visibility}"/>
     <!-- BACK SENSOR -->
     <joint name="back_tof_joint" type="fixed">
@@ -119,5 +114,4 @@
                                     name="back_tof"
                                     on="true"
-                                    visible="${front_back_sensor_visibility}"
-                                    material="${gazebo_tof_material}"/>
+                                    visible="${front_back_sensor_visibility}"/>
 </robot>

File: dev_ws/src/minirys_sim/description/variables.xacro (robot description, xacro)
@@ -3,34 +3,20 @@
     <xacro:property name="color_code_material" value="custom_color"/>
     <xacro:property name="batteries_material" value="purple"/>
-    <xacro:property name="gazebo_batteries_material" value="rys/purple"/>
     <!-- MATERIALS -->
         <!-- WHEEL -->
         <xacro:property name="tire_material" value="${color_code_material}"/>
         <xacro:property name="wheel_material" value="black"/>
-        <xacro:property name="gazebo_wheel_material" value="rys/black"/>
     <!-- SENSORS -->
         <!-- TOF -->
             <xacro:property name="tof_material" value="dark_red"/>
-            <xacro:property name="gazebo_tof_material" value="rys/red"/>
         <!-- CAMERA -->
-            <xacro:property name="camera_base_material" value="dark_grey"/>
+            <xacro:property name="camera_base_material" value="dark_gray"/>
             <xacro:property name="camera_PCB_material" value="black"/>
             <xacro:property name="camera_bumper_material" value="${color_code_material}"/>
             <xacro:property name="camera_lens_material" value="lens"/>
-            <xacro:property name="gazebo_camera_base_material" value="rys/dark_gray"/>
-            <xacro:property name="gazebo_camera_PCB_material" value="rys/black"/>
-            <xacro:property name="gazebo_camera_lens_material" value="rys/lens"/>
     <!-- CHASSIS -->
         <xacro:property name="skeleton_material" value="black"/>
         <xacro:property name="fronts_material" value="${color_code_material}"/>
-        <xacro:property name="internal_components_material" value="grey"/>
-        <xacro:property name="gazebo_skeleton_material" value="rys/black"/>
-        <xacro:property name="gazebo_internal_components_material" value="rys/light_gray"/>
-        <xacro:if value="$(arg camera_enabled)">
-            <xacro:property name="label_hight" value="0.19"/>
-        </xacro:if>
-        <xacro:unless value="$(arg camera_enabled)">
-            <xacro:property name="label_hight" value="0.16"/>
-        </xacro:unless>
+        <xacro:property name="internal_components_material" value="gray"/>
     <!-- VARIABLES -->
         <!-- ROBOT STRUCTURE -->
@@ -38,4 +24,10 @@
             <xacro:property name="wheel_radius" value="0.056"/>
             <xacro:property name="wheel_width" value="0.0145"/>
+            <xacro:if value="$(arg camera_enabled)">
+                <xacro:property name="label_hight" value="0.19"/>
+            </xacro:if>
+            <xacro:unless value="$(arg camera_enabled)">
+                <xacro:property name="label_hight" value="0.16"/>
+            </xacro:unless>
         <!-- SENSORS -->
             <xacro:if value="$(arg horizontal_sensor_visibility)">
@@ -56,11 +48,10 @@
                 <xacro:property name="front_back_sensor_visibility" value="true"/>
             </xacro:if>
-            <!-- <xacro:unless value="$(arg all_sensor_visibility)"></xacro:unless> -->
-            <xacro:if value="$(arg none_sensor_visibility)">
+            <xacro:unless value="$(arg all_sensor_visibility)">
                 <xacro:property name="up_down_sensor_visibility" value="false"/>
                 <xacro:property name="right_left_sensor_visibility" value="false"/>
                 <xacro:property name="front_back_sensor_visibility" value="false"/>
-            </xacro:if>
-            <!-- <xacro:unless value="$(arg none_sensor_visibility)"></xacro:unless> -->
+            </xacro:unless>
+            <!-- <xacro:unless value="$(arg all_sensor_visibility)"></xacro:unless> -->
     <!-- FILE PATHS -->
         <!-- GAZEBOMATERIALS -->
